File: kicad_input/reference-design.kicad_pcb (KiCad board)
At the start: 2 copper layers, 104 x 83.9 mm, 30 parts

Commit message: new input design
Parts:
- removed Sensor_Driver1: TLC59108IRGYR, TLC59208FIRGYR:RGY16_2P55X2P05
- removed TP1: col0, TestPoint:TestPoint_Pad_2.0x2.0mm
- removed TP2: col1, TestPoint:TestPoint_Pad_2.0x2.0mm
- removed TP3: col2, TestPoint:TestPoint_Pad_2.0x2.0mm
- removed TP4: col3, TestPoint:TestPoint_Pad_2.0x2.0mm
- removed TP5: row0, TestPoint:TestPoint_Pad_2.0x2.0mm
- removed TP6: row1, TestPoint:TestPoint_Pad_2.0x2.0mm
- removed TP7: row2, TestPoint:TestPoint_Pad_2.0x2.0mm
- removed TP8: row3, TestPoint:TestPoint_Pad_2.0x2.0mm
- removed TP9: GND, TestPoint:TestPoint_Pad_2.0x2.0mm
- added C3: 2uF, Capacitor_SMD:C_0603_1608Metric, F.Cu at (16.0, 57.5)
- added C4: 2uF, Capacitor_SMD:C_0603_1608Metric, F.Cu at (16.0, 60.0)
- added GPIO1: TLA2528IRTER, TLA2528IRTER:WQFN16_RTE_TEX, F.Cu at (23.2, 67.5)
- added MOSFET1: SI2342DS-T1-GE3, SI2342DS-T1-GE3:SOT-23_TO-236_VIS, F.Cu at (30.8, 53.0)
- added MOSFET2: SI2342DS-T1-GE3, SI2342DS-T1-GE3:SOT-23_TO-236_VIS, F.Cu at (30.8, 58.0)
- added MOSFET3: SI2342DS-T1-GE3, SI2342DS-T1-GE3:SOT-23_TO-236_VIS, F.Cu at (30.8, 63.0)
- added MOSFET4: SI2342DS-T1-GE3, SI2342DS-T1-GE3:SOT-23_TO-236_VIS, F.Cu at (30.8, 68.0)
- added R1: 11K, Resistor_SMD:R_0603_1608Metric, F.Cu at (21.2, 52.5)
- added R2: DNP, Resistor_SMD:R_0603_1608Metric, F.Cu at (21.2, 55.0)
- added R3: 0, Resistor_SMD:R_0603_1608Metric, F.Cu at (21.2, 57.5)
- added R4: DNP, Resistor_SMD:R_0603_1608Metric, F.Cu at (21.2, 60.1)
- C1, C2: footprint Capacitor_SMD:C_0805_2012Metric_Pad1.18x1.45mm_HandSolder -> Capacitor_SMD:C_0603_1608Metric
- H11, H12, H15, H16, H3, H4, H7, H8: footprint AH49FNTR_G1:SC59_DIO_KeyswitchOutline -> AH49FNTR_G1:SC59_DIO_KeyswitchOutline_NoRuleArea
- moved C2 11.3 mm to (16.0, 55.0), turned to 0 degrees
- moved C1 5.22 mm to (16.0, 52.5), turned to 0 degrees
- moved ADC1 3.62 mm to (26.5, 42.8), turned to 0 degrees
- moved MCU1 3.47 mm to (24.4, 24.2)
Connections:
- net row0 renamed Net-(H1-VCC)
- net row1 renamed Net-(H5-VCC)
- net row2 renamed Net-(H10-VCC)
- net row3 renamed Net-(H13-VCC)
- ADC1 pad 11: GND -> Net-(ADC1-ADDR)
- C1 pad 1: +3.3V -> Net-(GPIO1-DECAP)
- C2 pad 1: Net-(ADC1-DECAP) -> +3.3V
Routing:
- net Net-(H5-VCC): track 140.2 -> 81.9 mm, vias 2 -> 0
- net +3.3V: track 80.3 -> 133.4 mm
- net col1: track 172.1 -> 125.2 mm, vias 7 -> 5
- net Net-(H10-VCC): track 122.4 -> 76.0 mm, vias 2 -> 0
- net col0: track 190.5 -> 145.4 mm, vias 8 -> 3
- net Net-(H13-VCC): track 124.7 -> 81.4 mm, vias 3 -> 0
- net Net-(H1-VCC): track 140.3 -> 98.5 mm, vias 3 -> 2
- net col2: track 149.5 -> 109.1 mm
- net i2c0_scl: track 46.6 -> 75.1 mm, vias 1 -> 3
- net Net-(ADC1-ADDR): track 0.00 -> 27.4 mm, vias 0 -> 2
- net col3: track 119.4 -> 92.4 mm, vias 4 -> 7
- net i2c0_sda: track 44.8 -> 71.1 mm
- net Net-(GPIO1-DECAP): track 0.00 -> 23.4 mm, vias 0 -> 2
- net GND: track 422.0 -> 401.3 mm, vias 5 -> 7
- net Net-(GPIO1-ADDR): track 0.00 -> 20.6 mm, vias 0 -> 2
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Other:
- board text added: "ParaKeyt Reference r0.9 UMass ECE SDP26 Team 32 Bennett Gilig, Raffi Belorian, Rikhav Shah, Shlok Raval, Theo Krueger. THIS SIDE FACE DOWN"
- board text removed: "ParaKeyt Reference r0.8 UMass ECE SDP26 Team 32 Bennett Gilig, Raffi Belorian, Rikhav Shah, Shlok Raval, Theo Krueger. THIS SIDE FACE DOWN"
- board text removed: "Some areas intentionally have a filled/unfilled zone for interference tests"

Commit message: good working case generation
Parts:
- removed ADC1, GPIO1: TLA2528IRTER, TLA2528IRTER:WQFN16_RTE_TEX
- removed C1, C2, C3, C4: 2uF, Capacitor_SMD:C_0603_1608Metric
- removed H1, H10, H11, H12, H13, H14, H15, H16, H2, H3, H4, H5, H6, H7, H8, H9: AH49FNTR-G1, AH49FNTR_G1:SC59_DIO_KeyswitchOutline_NoRuleArea
- removed MCU1: RP2040-Zero, RP2040-Zero:rp2040-zero-tht
- removed MOSFET1, MOSFET2, MOSFET3, MOSFET4: SI2342DS-T1-GE3, SI2342DS-T1-GE3:SOT-23_TO-236_VIS
- removed R1: 11K, Resistor_SMD:R_0603_1608Metric
- removed R2, R4: DNP, Resistor_SMD:R_0603_1608Metric
- removed R3: 0, Resistor_SMD:R_0603_1608Metric
- added REF**: SC59_DIO_KeyswitchOutline_NoRuleArea_mosfet, SC59_DIO_KeyswitchOutline_NoRuleArea_mosfet, F.Cu at (9.53, 9.53)
- added REF**: SC59_DIO_KeyswitchOutline_NoRuleArea_mosfet, SC59_DIO_KeyswitchOutline_NoRuleArea, F.Cu at (181.0, 9.53)
- added REF**: SC59_DIO_KeyswitchOutline_NoRuleArea_mosfet, SC59_DIO_KeyswitchOutline_NoRuleArea, F.Cu at (200.0, 9.53)
- added REF**: SC59_DIO_KeyswitchOutline_NoRuleArea_mosfet, SC59_DIO_KeyswitchOutline_NoRuleArea, F.Cu at (219.1, 9.53)
- added REF**: SC59_DIO_KeyswitchOutline_NoRuleArea_mosfet, SC59_DIO_KeyswitchOutline_NoRuleArea, F.Cu at (238.1, 9.53)
- added REF**: SC59_DIO_KeyswitchOutline_NoRuleArea_mosfet, SC59_DIO_KeyswitchOutline_NoRuleArea, F.Cu at (257.2, 9.53)
- added REF**: SC59_DIO_KeyswitchOutline_NoRuleArea_mosfet, SC59_DIO_KeyswitchOutline_NoRuleArea, F.Cu at (9.53, 28.6)
- added REF**: SC59_DIO_KeyswitchOutline_NoRuleArea_mosfet, SC59_DIO_KeyswitchOutline_NoRuleArea, F.Cu at (33.3, 28.6)
- added REF**: SC59_DIO_KeyswitchOutline_NoRuleArea_mosfet, SC59_DIO_KeyswitchOutline_NoRuleArea_mosfet, F.Cu at (52.4, 28.6)
- added REF**: SC59_DIO_KeyswitchOutline_NoRuleArea_mosfet, SC59_DIO_KeyswitchOutline_NoRuleArea, F.Cu at (71.4, 28.6)
- added REF**: SC59_DIO_KeyswitchOutline_NoRuleArea_mosfet, SC59_DIO_KeyswitchOutline_NoRuleArea, F.Cu at (90.5, 28.6)
- added REF**: SC59_DIO_KeyswitchOutline_NoRuleArea_mosfet, SC59_DIO_KeyswitchOutline_NoRuleArea, F.Cu at (28.6, 9.53)
- added REF**: SC59_DIO_KeyswitchOutline_NoRuleArea_mosfet, SC59_DIO_KeyswitchOutline_NoRuleArea, F.Cu at (109.5, 28.6)
- added REF**: SC59_DIO_KeyswitchOutline_NoRuleArea_mosfet, SC59_DIO_KeyswitchOutline_NoRuleArea, F.Cu at (128.6, 28.6)
- added REF**: SC59_DIO_KeyswitchOutline_NoRuleArea_mosfet, SC59_DIO_KeyswitchOutline_NoRuleArea, F.Cu at (147.6, 28.6)
- added REF**: SC59_DIO_KeyswitchOutline_NoRuleArea_mosfet, SC59_DIO_KeyswitchOutline_NoRuleArea, F.Cu at (166.7, 28.6)
- added REF**: SC59_DIO_KeyswitchOutline_NoRuleArea_mosfet, SC59_DIO_KeyswitchOutline_NoRuleArea, F.Cu at (185.7, 28.6)
- added REF**: SC59_DIO_KeyswitchOutline_NoRuleArea_mosfet, SC59_DIO_KeyswitchOutline_NoRuleArea_mosfet, F.Cu at (204.8, 28.6)
- added REF**: SC59_DIO_KeyswitchOutline_NoRuleArea_mosfet, SC59_DIO_KeyswitchOutline_NoRuleArea, F.Cu at (223.8, 28.6)
- added REF**: SC59_DIO_KeyswitchOutline_NoRuleArea_mosfet, SC59_DIO_KeyswitchOutline_NoRuleArea, F.Cu at (242.9, 28.6)
- added REF**: SC59_DIO_KeyswitchOutline_NoRuleArea_mosfet, SC59_DIO_KeyswitchOutline_NoRuleArea, F.Cu at (261.9, 28.6)
- added REF**: SC59_DIO_KeyswitchOutline_NoRuleArea_mosfet, SC59_DIO_KeyswitchOutline_NoRuleArea, F.Cu at (9.53, 47.6)
- added REF**: SC59_DIO_KeyswitchOutline_NoRuleArea_mosfet, SC59_DIO_KeyswitchOutline_NoRuleArea, F.Cu at (47.6, 9.53)
- added REF**: SC59_DIO_KeyswitchOutline_NoRuleArea_mosfet, SC59_DIO_KeyswitchOutline_NoRuleArea, F.Cu at (38.1, 47.6)
- added REF**: SC59_DIO_KeyswitchOutline_NoRuleArea_mosfet, SC59_DIO_KeyswitchOutline_NoRuleArea, F.Cu at (57.2, 47.6)
- added REF**: SC59_DIO_KeyswitchOutline_NoRuleArea_mosfet, SC59_DIO_KeyswitchOutline_NoRuleArea, F.Cu at (76.2, 47.6)
- added REF**: SC59_DIO_KeyswitchOutline_NoRuleArea_mosfet, SC59_DIO_KeyswitchOutline_NoRuleArea_mosfet, F.Cu at (95.2, 47.6)
- added REF**: SC59_DIO_KeyswitchOutline_NoRuleArea_mosfet, SC59_DIO_KeyswitchOutline_NoRuleArea, F.Cu at (114.3, 47.6)
- added REF**: SC59_DIO_KeyswitchOutline_NoRuleArea_mosfet, SC59_DIO_KeyswitchOutline_NoRuleArea, F.Cu at (133.3, 47.6)
- added REF**: SC59_DIO_KeyswitchOutline_NoRuleArea_mosfet, SC59_DIO_KeyswitchOutline_NoRuleArea, F.Cu at (152.4, 47.6)
- added REF**: SC59_DIO_KeyswitchOutline_NoRuleArea_mosfet, SC59_DIO_KeyswitchOutline_NoRuleArea, F.Cu at (171.5, 47.6)
- added REF**: SC59_DIO_KeyswitchOutline_NoRuleArea_mosfet, SC59_DIO_KeyswitchOutline_NoRuleArea, F.Cu at (190.5, 47.6)
- added REF**: SC59_DIO_KeyswitchOutline_NoRuleArea_mosfet, SC59_DIO_KeyswitchOutline_NoRuleArea, F.Cu at (209.6, 47.6)
- added REF**: SC59_DIO_KeyswitchOutline_NoRuleArea_mosfet, SC59_DIO_KeyswitchOutline_NoRuleArea, F.Cu at (66.7, 9.53)
- added REF**: SC59_DIO_KeyswitchOutline_NoRuleArea_mosfet, SC59_DIO_KeyswitchOutline_NoRuleArea, F.Cu at (228.6, 47.6)
- added REF**: SC59_DIO_KeyswitchOutline_NoRuleArea_mosfet, SC59_DIO_KeyswitchOutline_NoRuleArea_mosfet, F.Cu at (247.7, 47.6)
- added REF**: SC59_DIO_KeyswitchOutline_NoRuleArea_mosfet, SC59_DIO_KeyswitchOutline_NoRuleArea, F.Cu at (9.53, 66.7)
- added REF**: SC59_DIO_KeyswitchOutline_NoRuleArea_mosfet, SC59_DIO_KeyswitchOutline_NoRuleArea, F.Cu at (42.9, 66.7)
- added REF**: SC59_DIO_KeyswitchOutline_NoRuleArea_mosfet, SC59_DIO_KeyswitchOutline_NoRuleArea, F.Cu at (61.9, 66.7)
- added REF**: SC59_DIO_KeyswitchOutline_NoRuleArea_mosfet, SC59_DIO_KeyswitchOutline_NoRuleArea, F.Cu at (81.0, 66.7)
- added REF**: SC59_DIO_KeyswitchOutline_NoRuleArea_mosfet, SC59_DIO_KeyswitchOutline_NoRuleArea, F.Cu at (100.0, 66.7)
- added REF**: SC59_DIO_KeyswitchOutline_NoRuleArea_mosfet, SC59_DIO_KeyswitchOutline_NoRuleArea, F.Cu at (119.1, 66.7)
- added REF**: SC59_DIO_KeyswitchOutline_NoRuleArea_mosfet, SC59_DIO_KeyswitchOutline_NoRuleArea, F.Cu at (138.1, 66.7)
- added REF**: SC59_DIO_KeyswitchOutline_NoRuleArea_mosfet, SC59_DIO_KeyswitchOutline_NoRuleArea_mosfet, F.Cu at (157.2, 66.7)
- added REF**: SC59_DIO_KeyswitchOutline_NoRuleArea_mosfet, SC59_DIO_KeyswitchOutline_NoRuleArea, F.Cu at (85.7, 9.53)
- added REF**: SC59_DIO_KeyswitchOutline_NoRuleArea_mosfet, SC59_DIO_KeyswitchOutline_NoRuleArea, F.Cu at (176.2, 66.7)
- added REF**: SC59_DIO_KeyswitchOutline_NoRuleArea_mosfet, SC59_DIO_KeyswitchOutline_NoRuleArea, F.Cu at (195.3, 66.7)
- added REF**: SC59_DIO_KeyswitchOutline_NoRuleArea_mosfet, SC59_DIO_KeyswitchOutline_NoRuleArea, F.Cu at (214.3, 66.7)
- added REF**: SC59_DIO_KeyswitchOutline_NoRuleArea_mosfet, SC59_DIO_KeyswitchOutline_NoRuleArea, F.Cu at (233.4, 66.7)
- added REF**: SC59_DIO_KeyswitchOutline_NoRuleArea_mosfet, SC59_DIO_KeyswitchOutline_NoRuleArea, F.Cu at (9.53, 85.7)
- added REF**: SC59_DIO_KeyswitchOutline_NoRuleArea_mosfet, SC59_DIO_KeyswitchOutline_NoRuleArea, F.Cu at (33.3, 85.7)
- added REF**: SC59_DIO_KeyswitchOutline_NoRuleArea_mosfet, SC59_DIO_KeyswitchOutline_NoRuleArea, F.Cu at (52.4, 85.7)
- added REF**: SC59_DIO_KeyswitchOutline_NoRuleArea_mosfet, SC59_DIO_KeyswitchOutline_NoRuleArea_mosfet, F.Cu at (76.2, 85.7)
- added REF**: SC59_DIO_KeyswitchOutline_NoRuleArea_mosfet, SC59_DIO_KeyswitchOutline_NoRuleArea, F.Cu at (195.3, 85.7)
- added REF**: SC59_DIO_KeyswitchOutline_NoRuleArea_mosfet, SC59_DIO_KeyswitchOutline_NoRuleArea, F.Cu at (219.1, 85.7)
- added REF**: SC59_DIO_KeyswitchOutline_NoRuleArea_mosfet, SC59_DIO_KeyswitchOutline_NoRuleArea, F.Cu at (104.8, 9.53)
- added REF**: SC59_DIO_KeyswitchOutline_NoRuleArea_mosfet, SC59_DIO_KeyswitchOutline_NoRuleArea, F.Cu at (238.1, 85.7)
- added REF**: SC59_DIO_KeyswitchOutline_NoRuleArea_mosfet, SC59_DIO_KeyswitchOutline_NoRuleArea, F.Cu at (257.2, 85.7)
- added REF**: WQFN16_RTE_TEX_with_caps_and_Rs, WQFN16_RTE_TEX_with_caps_and_Rs, F.Cu at (21.0, 21.0)
- added REF**: WQFN16_RTE_TEX_with_caps_and_Rs, WQFN16_RTE_TEX_with_caps_and_Rs, F.Cu at (21.0, 32.4)
- added REF**: SC59_DIO_KeyswitchOutline_NoRuleArea_mosfet, SC59_DIO_KeyswitchOutline_NoRuleArea, F.Cu at (123.8, 9.53)
- added REF**: SC59_DIO_KeyswitchOutline_NoRuleArea_mosfet, SC59_DIO_KeyswitchOutline_NoRuleArea, F.Cu at (142.9, 9.53)
- added REF**: SC59_DIO_KeyswitchOutline_NoRuleArea_mosfet, SC59_DIO_KeyswitchOutline_NoRuleArea_mosfet, F.Cu at (161.9, 9.53)
- added U?: rp2040-zero-tht, rp2040-zero-tht, F.Cu at (305.7, 12.8)
Routing:
- net GND: track 401.3 -> 0.00 mm, vias 7 -> 0
- net col0: track 145.4 -> 0.00 mm, vias 3 -> 0
- net +3.3V: track 133.4 -> 0.00 mm, vias 3 -> 0
- net col1: track 125.2 -> 0.00 mm, vias 5 -> 0
- net col2: track 109.1 -> 0.00 mm, vias 5 -> 0
- net Net-(H1-VCC): track 98.5 -> 0.00 mm, vias 2 -> 0
- net col3: track 92.4 -> 0.00 mm, vias 7 -> 0
- net Net-(H5-VCC): track 81.9 -> 0.00 mm
- net Net-(H13-VCC): track 81.4 -> 0.00 mm
- net Net-(H10-VCC): track 76.0 -> 0.00 mm
- net i2c0_scl: track 75.1 -> 0.00 mm, vias 3 -> 0
- net i2c0_sda: track 71.1 -> 0.00 mm, vias 2 -> 0
- net Net-(ADC1-ADDR): track 27.4 -> 0.00 mm, vias 2 -> 0
- net Net-(ADC1-DECAP): track 24.4 -> 0.00 mm, vias 2 -> 0
- net Net-(GPIO1-DECAP): track 23.4 -> 0.00 mm, vias 2 -> 0
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- removed copper zone on B.Cu, net GND
- removed copper zone on F.Cu, net GND
Other:
- board size 104 x 83.9 mm -> 323.9 x 95.2 mm
- rule pad_to_mask_clearance: 0 -> 0.0
- board text removed: "ParaKeyt Reference r0.9 UMass ECE SDP26 Team 32 Bennett Gilig, Raffi Belorian, Rikhav Shah, Shlok Raval, Theo Krueger. THIS SIDE FACE DOWN"
